File: hardware/minipc-power.kicad_sch (KiCad schematic)
At the start: 106 parts, among them J1 USB-C HRO TYPE-C-31-M-12, J10 VSYS (switch), J11 CHG, J12 PG_CHG, J13 VBAT_SENSE, J14 3V3_PG, J15 GND, J16 GND, J17 GND, J2 BAT+, J3 BAT-, J4 NTC, J5 NTC-, J6 +12V OUT, J7 +5V OUT, J8 +3V3 OUT, J9 EN (switch), Q1 CSD13202Q2, Q2 CSD13202Q2, Q3 CSD13202Q2, Q4 CSD25404Q3, Q5 CSD25404Q3, Q6 2N7002, U1 CH224Q, U2 BQ25606, U3 HY2113-MB1A, U4 TPS61178, U5 TPS61088-Q1, U6 TPS63802

Commit message: Protection FETs: DMN1004UFV, block re-laid out with B.Cu copper; heat 5.0 -> 3.4 W at 15 W
Q1-Q3 CSD13202Q2 (8.4 mOhm at 3 V) -> Diodes DMN1004UFV (C316138, 3.2 / 5.1 mOhm at 2.5 V, PowerDI3333-8;
KiCad Diodes_PowerDI3333-8 checked against the datasheet's suggested pads; JLCImport 3D model, orientation checked
by the pin-1 dot). FET loss at 15 W from an empty cell 1.72 -> 0.53 W, board 5.0 -> 3.4 W (docs/thermal.md).
The 3.3 mm parts no longer fit in a row: Q2 | Q1 face across the CELLN gap, Q1's drain at J3, Q3 under Q2's drain;
U3 between Q3 and H2's keep-out, R7-R10 / C8 under J3. Same-net B.Cu islands joined by vias; OD, CS and Q1's gate
take short B.Cu lanes. U3 stays HY2113-MB1A: its FET-sensed trip moves to ~18-46 A (power-design s3).
A Vishay SiSS80DN was chosen first and dropped: stocked on LCSC China only, not for JLCPCB global assembly.

routing.via_near: no via on any pad but the one it stitches (two had landed in Q3's neighbouring source pads).
docs/review_config.json: the review's power runs, updated for the new pins and net names.
skill-gaps.md 46-52. DRC 0, ERC 0, unconnected 0, parity 0, board_lint 0, pin decisions and part fields clean;
bom_check (global) 0 problems. hardware/production/ still predates this board.
Parts:
- Q1, Q2, Q3: value CSD13202Q2 -> DMN1004UFV; footprint Package_SON:Texas_DQK -> Package_SON:Diodes_PowerDI3333-8; symbol minipc:CSD13202Q2 -> minipc:DMN1004UFV; LCSC C187839 -> C316138
Connections:
- net GND: now also Q3.1 (S), Q3.2 (S), Q3.3 (S); no longer Q3.4 (S), Q3.7 (S)
- net at U3.1 (OD): now also Q2.4 (G); no longer Q2.3 (G)
- net at U3.3 (OC): now also Q3.4 (G); no longer Q3.3 (G)
- net at R10.1, R9.2: now also Q1.4 (G); no longer Q1.3 (G)
- new net: C8.2, Q1.1 (S), Q1.2 (S), Q1.3 (S), Q2.1 (S), Q2.2 (S), Q2.3 (S), R10.2, U3.6 (VSS)
- new net: Q2.5 (D), Q3.5 (D)
- new net: J3.1, Q1.5 (D)
Other:
- note added: "Q1: a reversed pack turns it off and its body diode blocks, so U3 never sees reverse voltage. Trip: 250 mV / (Q2+Q3) = ~17 A hot ... ~45 A cold."
- note removed: "Q1: a reversed pack turns it off and its body diode blocks, so U3 never sees reverse voltage. Trip: 250 mV / (Q2+Q3) = ~8 A hot ... ~15 A cold."
Changed lines of the file:
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@@
 		)
 	)
-	(text "Q1: a reversed pack turns it off and its body diode\nblocks, so U3 never sees reverse voltage.\nTrip: 250 mV / (Q2+Q3) = ~8 A hot ... ~15 A cold."
+	(text "Q1: a reversed pack turns it off and its body diode\nblocks, so U3 never sees reverse voltage.\nTrip: 250 mV / (Q2+Q3) = ~17 A hot ... ~45 A cold."
 		(exclude_from_sim no)
 		(at 345.44 167.64 0)
@@
 	)
 	(symbol
-		(lib_id "minipc:CSD13202Q2")
+		(lib_id "minipc:DMN1004UFV")
 		(at 365.76 137.16 90)
 		(unit 1)
@@
 			)
 		)
-		(property "Value" "CSD13202Q2"
+		(property "Value" "DMN1004UFV"
 			(at 370.84 127 90)
 			(show_name no)
@@
 			)
 		)
-		(property "Footprint" "Package_SON:Texas_DQK"
+		(property "Footprint" "Package_SON:Diodes_PowerDI3333-8"
 			(at 365.76 137.16 90)
 			(hide yes)
@@
 			)
 		)
-		(property "Datasheet" "https://www.ti.com/lit/ds/symlink/csd13202q2.pdf"
+		(property "Datasheet" "https://www.diodes.com/assets/Datasheets/DMN1004UFV.pdf"
 			(at 365.76 137.16 90)
 			(hide yes)
@@
 			)
 		)
-		(property "Description" "12 V N-FET, TI DQK (KiCad Package_SON:Texas_DQK pads)"
+		(property "Description" "12 V N-FET, 2.5 V rated, Diodes PowerDI3333-8 type UX (KiCad Diodes_PowerDI3333-8 pads)"
 			(at 365.76 137.16 90)
 			(hide yes)
@@
 			)
 		)
-		(property "LCSC" "C187839"
+		(property "LCSC" "C316138"
 			(at 365.76 137.16 90)
 			(hide yes)
@@
 			)
 		)
-		(pin "1"
-		)
-		(pin "2"
-		)
 		(pin "5"
 		)
-		(pin "6"
-		)
-		(pin "8"
+		(pin "4"
 		)
-		(pin "3"
+		(pin "1"
 		)
-		(pin "4"
+		(pin "2"
 		)
-		(pin "7"
+		(pin "3"
 		)
 		(instances
@@
 	)
 	(symbol
-		(lib_id "minipc:CSD13202Q2")
+		(lib_id "minipc:DMN1004UFV")
 		(at 396.24 132.08 270)
 		(unit 1)
@@
 			)
 		)
-		(property "Value" "CSD13202Q2"
+		(property "Value" "DMN1004UFV"
 			(at 391.16 144.78 90)
 			(show_name no)
@@
 			)
 		)
-		(property "Footprint" "Package_SON:Texas_DQK"
+		(property "Footprint" "Package_SON:Diodes_PowerDI3333-8"
 			(at 396.24 132.08 90)
 			(hide yes)
@@
 			)
 		)
-		(property "Datasheet" "https://www.ti.com/lit/ds/symlink/csd13202q2.pdf"
+		(property "Datasheet" "https://www.diodes.com/assets/Datasheets/DMN1004UFV.pdf"
 			(at 396.24 132.08 90)
 			(hide yes)
@@
 			)
 		)
-		(property "Description" "12 V N-FET, TI DQK (KiCad Package_SON:Texas_DQK pads)"
+		(property "Description" "12 V N-FET, 2.5 V rated, Diodes PowerDI3333-8 type UX (KiCad Diodes_PowerDI3333-8 pads)"
 			(at 396.24 132.08 90)
 			(hide yes)
@@
 			)
 		)
-		(property "LCSC" "C187839"
+		(property "LCSC" "C316138"
 			(at 396.24 132.08 90)
 			(hide yes)
@@
 			)
 		)
-		(pin "1"
-		)
-		(pin "2"
-		)
 		(pin "5"
 		)
-		(pin "6"
-		)
-		(pin "8"
+		(pin "4"
 		)
-		(pin "3"
+		(pin "1"
 		)
-		(pin "4"
+		(pin "2"
 		)
-		(pin "7"
+		(pin "3"
 		)
 		(instances
@@
 	)
 	(symbol
-		(lib_id "minipc:CSD13202Q2")
+		(lib_id "minipc:DMN1004UFV")
 		(at 416.56 132.08 90)
 		(mirror x)
@@
 			)
 		)
-		(property "Value" "CSD13202Q2"
+		(property "Value" "DMN1004UFV"
 			(at 420.37 129.54 90)
 			(show_name no)
@@
 			)
 		)
-		(property "Footprint" "Package_SON:Texas_DQK"
+		(property "Footprint" "Package_SON:Diodes_PowerDI3333-8"
 			(at 416.56 132.08 90)
 			(hide yes)
@@
 			)
 		)
-		(property "Datasheet" "https://www.ti.com/lit/ds/symlink/csd13202q2.pdf"
+		(property "Datasheet" "https://www.diodes.com/assets/Datasheets/DMN1004UFV.pdf"
 			(at 416.56 132.08 90)
 			(hide yes)
@@
 			)
 		)
-		(property "Description" "12 V N-FET, TI DQK (KiCad Package_SON:Texas_DQK pads)"
+		(property "Description" "12 V N-FET, 2.5 V rated, Diodes PowerDI3333-8 type UX (KiCad Diodes_PowerDI3333-8 pads)"
 			(at 416.56 132.08 90)
 			(hide yes)
@@
 			)
 		)
-		(property "LCSC" "C187839"
+		(property "LCSC" "C316138"
 			(at 416.56 132.08 90)
 			(hide yes)
@@
 			)
 		)
-		(pin "1"
-		)
-		(pin "2"
-		)
 		(pin "5"
 		)
-		(pin "6"
-		)
-		(pin "8"
+		(pin "4"
 		)
-		(pin "3"
+		(pin "1"
 		)
-		(pin "4"
+		(pin "2"
 		)
-		(pin "7"
+		(pin "3"
 		)
 		(instances
